Commit message: added realsense depth camera to wheelchair

File: src/intellwheels_desc/urdf/rplidar.gazebo.xacro (robot description, xacro)
@@ -1,5 +1,5 @@
 <?xml version="1.0"?>
 <robot xmlns:xacro="http://www.ros.org/wiki/xacro">
-	<xacro:macro name="rplidar" params="prefix">
+	<xacro:macro name="rplidar_sensor" params="prefix">
 		<gazebo reference="${prefix}_rplidar_link">
 			<sensor name="${prefix}_rplidar" type="ray">
@@ -33,5 +33,5 @@
 		</gazebo>
 	</xacro:macro>
-	<xacro:rplidar prefix="left_front"/>
-	<xacro:rplidar prefix="right_back"/>
+	<xacro:rplidar_sensor prefix="left_front"/>
+	<xacro:rplidar_sensor prefix="right_back"/>
 </robot>

File: src/intellwheels_desc/urdf/wheelchair.urdf.xacro (robot description, xacro)
@@ -10,4 +10,5 @@
 	<xacro:include filename="${urdf}/drive_wheel.urdf.xacro"/>
 	<xacro:include filename="${urdf}/rplidar.urdf.xacro"/>
+	<xacro:include filename="${urdf}/realsense.urdf.xacro"/>
 	<!-- build wheelchair -->
 	<xacro:base/>
@@ -20,7 +21,10 @@
 	<xacro:rplidar prefix="left_front"/>
 	<xacro:rplidar prefix="right_back" right="1" back="1"/>
+	<xacro:realsense prefix="right_front" right="1"/>
+	<xacro:realsense prefix="left_back" back="1"/>
 	<!-- import gazebo stuff: controllers, materials, sensors, etc... -->
 	<xacro:include filename="${urdf}/materials.gazebo.xacro"/>
 	<xacro:include filename="${urdf}/diff_drive.gazebo.xacro"/>
 	<xacro:include filename="${urdf}/rplidar.gazebo.xacro"/>
+	<xacro:include filename="${urdf}/realsense.gazebo.xacro"/>
 </robot>
