Commit message: navigation now uses depth cam instead of lidars

File: src/intellwheels_desc/urdf/diff_drive.gazebo.xacro (robot description, xacro)
@@ -1,25 +1,27 @@
 <?xml version="1.0"?>
 <robot xmlns:xacro="http://www.ros.org/wiki/xacro">
-	<gazebo>
-		<plugin name="differential_drive_controller" filename="libgazebo_ros_diff_drive.so">
-			<updateRate>100</updateRate>
-			<leftJoint>left_drive_wheel_joint</leftJoint>
-			<rightJoint>right_drive_wheel_joint</rightJoint>
-			<wheelSeparation>0.78</wheelSeparation>
-			<wheelDiameter>0.42</wheelDiameter>
-			<wheelAcceleration>1</wheelAcceleration>
-			<wheelTorque>20</wheelTorque>
-			<commandTopic>cmd_vel</commandTopic>
-			<odometryTopic>odom</odometryTopic>
-			<odometryFrame>odom</odometryFrame>
-			<robotBaseFrame>base_footprint</robotBaseFrame>
-			<odometrySource>world</odometrySource>
-			<publishWheelTF>false</publishWheelTF>
-			<publishOdomTF>true</publishOdomTF>
-			<publishWheelJointState>false</publishWheelJointState>
-			<legacyMode>false</legacyMode>
-			<rosDebugLevel>na</rosDebugLevel>
-			<publishTf>true</publishTf>
-		</plugin>
-	</gazebo>
+	<xacro:macro name="diff_drive_controller">
+		<gazebo>
+			<plugin name="differential_drive_controller" filename="libgazebo_ros_diff_drive.so">
+				<updateRate>100</updateRate>
+				<leftJoint>left_drive_wheel_joint</leftJoint>
+				<rightJoint>right_drive_wheel_joint</rightJoint>
+				<wheelSeparation>0.78</wheelSeparation>
+				<wheelDiameter>0.42</wheelDiameter>
+				<wheelAcceleration>1</wheelAcceleration>
+				<wheelTorque>20</wheelTorque>
+				<commandTopic>cmd_vel</commandTopic>
+				<odometryTopic>odom</odometryTopic>
+				<odometryFrame>odom</odometryFrame>
+				<robotBaseFrame>base_footprint</robotBaseFrame>
+				<odometrySource>world</odometrySource>
+				<publishWheelTF>false</publishWheelTF>
+				<publishOdomTF>true</publishOdomTF>
+				<publishWheelJointState>false</publishWheelJointState>
+				<legacyMode>false</legacyMode>
+				<rosDebugLevel>na</rosDebugLevel>
+				<publishTf>true</publishTf>
+			</plugin>
+		</gazebo>
+	</xacro:macro>
 </robot>

File: src/intellwheels_desc/urdf/materials.gazebo.xacro (robot description, xacro)
@@ -22,5 +22,3 @@
 		</gazebo>
 	</xacro:macro>
-	<xacro:drive_wheel_mat prefix="left"/>
-	<xacro:drive_wheel_mat prefix="right"/>
 </robot>

File: src/intellwheels_desc/urdf/realsense.gazebo.xacro (robot description, xacro)
@@ -1,13 +1,13 @@
 <?xml version="1.0"?>
 <robot xmlns:xacro="http://www.ros.org/wiki/xacro">
-	<xacro:macro name="realsense_sensor" params="prefix">
-		<gazebo reference="${prefix}_realsense_link">
-			<sensor name="${prefix}_realsense" type="depth">
+	<xacro:macro name="realsense_sensor">
+		<gazebo reference="realsense_link">
+			<sensor name="realsense" type="depth">
 				<update_rate>30</update_rate>
 				<camera>
 					<horizontal_fov>1.22</horizontal_fov>
 					<image>
-						<width>1024</width>
-						<height>768</height>
+						<width>640</width>
+						<height>480</height>
 					</image>
 					<clip>
@@ -16,7 +16,10 @@
 					</clip>
 				</camera>
-				<plugin name="${prefix}_realsense_controller" filename="libgazebo_ros_openni_kinect.so">
-					<baseline>0.2</baseline>
-					<cameraName>${prefix}_realsense</cameraName>
+				<plugin name="realsense_controller" filename="libgazebo_ros_openni_kinect.so">
+					<!-- used only for stereo cameras -->
+					<baseline>0</baseline>
+					<hackBaseline>0</hackBaseline>
+					<!-- topics and naming -->
+					<cameraName>realsense</cameraName>
 					<imageTopicName>color/image_raw</imageTopicName>
 					<cameraInfoTopicName>color/camera_info</cameraInfoTopicName>
@@ -24,5 +27,9 @@
 					<depthImageCameraInfoTopicName>depth/camera_info</depthImageCameraInfoTopicName>
 					<pointCloudTopicName>depth/points</pointCloudTopicName>
-					<frameName>${prefix}_realsense_optical_link</frameName>
+					<frameName>realsense_optical_link</frameName>
+					<!-- same clipping values as sensor -->
+					<pointCloudCutoff>0.25</pointCloudCutoff>
+					<pointCloudCutoffMax>9</pointCloudCutoffMax>
+					<!-- camera lens distortion -->
 					<distortionK1>0</distortionK1>
 					<distortionK2>0</distortionK2>
@@ -30,14 +37,12 @@
 					<distortionT1>0</distortionT1>
 					<distortionT2>0</distortionT2>
+					<!-- auto computed when set to 0 -->
 					<CxPrime>0</CxPrime>
 					<Cx>0</Cx>
 					<Cy>0</Cy>
 					<focalLength>0</focalLength>
-					<hackBaseline>0</hackBaseline>
 				</plugin>
 			</sensor>
 		</gazebo>
 	</xacro:macro>
-	<xacro:realsense_sensor prefix="right_front"/>
-	<xacro:realsense_sensor prefix="left_back"/>
 </robot>

File: src/intellwheels_desc/urdf/realsense.urdf.xacro (robot description, xacro)
@@ -1,10 +1,7 @@
 <?xml version="1.0"?>
 <robot xmlns:xacro="http://www.ros.org/wiki/xacro">
-	<!-- Intel RealSense LiDAR Camera L515 -->
-	<xacro:macro name="realsense" params="prefix right:=0 back:=0">
-		<xacro:property name="left" value="${1 - right}"/>
-		<xacro:property name="front" value="${1 - back}"/>
-		<link name="${prefix}_realsense_optical_link"/>
-		<link name="${prefix}_realsense_link">
+	<xacro:macro name="realsense">
+		<link name="realsense_optical_link"/>
+		<link name="realsense_support_link">
 			<inertial>
 				<mass value="1"/>
@@ -13,17 +10,34 @@
 			<visual>
 				<geometry>
+					<box size="0.01 0.1 0.3"/>
+				</geometry>
+			</visual>
+		</link>
+		<link name="realsense_link">
+			<inertial>
+				<mass value="1"/>
+				<xacro:insert_block name="default_inertia"/>
+			</inertial>
+			<visual>
+				<origin rpy="0 ${PI / 2} 0"/>
+				<geometry>
 					<cylinder radius="0.0305" length="0.026"/>
 				</geometry>
 			</visual>
 		</link>
-		<joint name="${prefix}_realsense_joint" type="fixed">
-			<origin xyz="${front * 0.435 - back * 0.485} ${left * 0.3 - right * 0.32} -0.15" rpy="0 0 ${back * PI}"/>
+		<joint name="realsense_support_joint" type="fixed">
+			<origin xyz="-0.6 0 1.15" rpy="0 0.2 0"/>
 			<parent link="base_link"/>
-			<child link="${prefix}_realsense_link"/>
+			<child link="realsense_support_link"/>
 		</joint>
-		<joint name="${prefix}_realsense_optical_joint" type="fixed">
+		<joint name="realsense_joint" type="fixed">
+			<origin xyz="0.01 0 0.1"/>
+			<parent link="realsense_support_link"/>
+			<child link="realsense_link"/>
+		</joint>
+		<joint name="realsense_optical_joint" type="fixed">
 			<origin rpy="${-PI / 2} 0 ${-PI / 2}"/>
-			<parent link="${prefix}_realsense_link"/>
-			<child link="${prefix}_realsense_optical_link"/>
+			<parent link="realsense_link"/>
+			<child link="realsense_optical_link"/>
 		</joint>
 	</xacro:macro>

File: src/intellwheels_desc/urdf/rplidar.gazebo.xacro (robot description, xacro)
@@ -4,5 +4,5 @@
 		<gazebo reference="${prefix}_rplidar_link">
 			<sensor name="${prefix}_rplidar" type="ray">
-				<visualize>true</visualize>
+				<visualize>false</visualize>
 				<update_rate>30</update_rate>
 				<ray>
@@ -33,5 +33,3 @@
 		</gazebo>
 	</xacro:macro>
-	<xacro:rplidar_sensor prefix="left_front"/>
-	<xacro:rplidar_sensor prefix="right_back"/>
 </robot>

File: src/intellwheels_desc/urdf/wheelchair.urdf.xacro (robot description, xacro)
@@ -21,6 +21,5 @@
 	<xacro:rplidar prefix="left_front"/>
 	<xacro:rplidar prefix="right_back" right="1" back="1"/>
-	<xacro:realsense prefix="right_front" right="1"/>
-	<xacro:realsense prefix="left_back" back="1"/>
+	<xacro:realsense/>
 	<!-- import gazebo stuff: controllers, materials, sensors, etc... -->
 	<xacro:include filename="${urdf}/materials.gazebo.xacro"/>
@@ -28,3 +27,10 @@
 	<xacro:include filename="${urdf}/rplidar.gazebo.xacro"/>
 	<xacro:include filename="${urdf}/realsense.gazebo.xacro"/>
+	<!-- build gazebo stuff -->
+	<xacro:diff_drive_controller/>
+	<xacro:drive_wheel_mat prefix="left"/>
+	<xacro:drive_wheel_mat prefix="right"/>
+	<xacro:rplidar_sensor prefix="left_front"/>
+	<xacro:rplidar_sensor prefix="right_back"/>
+	<xacro:realsense_sensor/>
 </robot>
