Commit message: added rplidar sensor

File: src/intellwheels_desc/urdf/base.urdf.xacro (robot description, xacro)
@@ -23,13 +23,13 @@
 			</visual>
 			<collision>
-				<origin xyz="-0.1 -0.02 0.55" rpy="0 -0.2 0"/>
+				<origin xyz="-0.1 -0.02 0.65" rpy="0 -0.2 0"/>
 				<geometry>
-					<box size="1.2 1.2 1.4"/>
+					<box size="1 1.2 1.4"/>
 				</geometry>
 			</collision>
 			<collision>
-				<origin xyz="0.59 0 -0.21" rpy="0 -0.1 0"/>
+				<origin xyz="0.59 0 -0.35" rpy="0 -0.1 0"/>
 				<geometry>
-					<box size="0.25 0.4 0.45"/>
+					<box size="0.25 0.4 0.2"/>
 				</geometry>
 			</collision>

File: src/intellwheels_desc/urdf/caster_arm.urdf.xacro (robot description, xacro)
@@ -21,7 +21,7 @@
 		</link>
 		<joint name="${prefix}_caster_arm_joint" type="continuous">
+			<origin xyz="${front * 0.435 - back * 0.485} ${left * 0.3 - right * 0.32} -0.24"/>
 			<parent link="base_link"/>
 			<child link="${prefix}_caster_arm_link"/>
-			<origin xyz="${front * 0.435 - back * 0.485} ${left * 0.3 - right * 0.32} -0.24"/>
 			<axis xyz="0 0 1"/>
 		</joint>

File: src/intellwheels_desc/urdf/wheelchair.urdf.xacro (robot description, xacro)
@@ -5,10 +5,9 @@
 	<xacro:include filename="${urdf}/common.urdf.xacro"/>
 	<xacro:include filename="${urdf}/base.urdf.xacro"/>
-	<xacro:include filename="${urdf}/base.gazebo.xacro"/>
 	<xacro:include filename="${urdf}/caster_arm.urdf.xacro"/>
 	<xacro:include filename="${urdf}/caster_wheel.urdf.xacro"/>
 	<xacro:include filename="${urdf}/caster.urdf.xacro"/>
 	<xacro:include filename="${urdf}/drive_wheel.urdf.xacro"/>
-	<xacro:include filename="${urdf}/drive_wheel.gazebo.xacro"/>
+	<xacro:include filename="${urdf}/rplidar.urdf.xacro"/>
 	<!-- build wheelchair -->
 	<xacro:base/>
@@ -19,5 +18,9 @@
 	<xacro:caster prefix="left_back" back="1"/>
 	<xacro:caster prefix="right_back" right="1" back="1"/>
-	<!-- import gazebo plugins: controllers, sensors, etc... -->
+	<xacro:rplidar prefix="left_front"/>
+	<xacro:rplidar prefix="right_back" right="1" back="1"/>
+	<!-- import gazebo stuff: controllers, materials, sensors, etc... -->
+	<xacro:include filename="${urdf}/materials.gazebo.xacro"/>
 	<xacro:include filename="${urdf}/diff_drive.gazebo.xacro"/>
+	<xacro:include filename="${urdf}/rplidar.gazebo.xacro"/>
 </robot>

Commit message: chair size is fixed. Need to clean urdfs afterwards and fix world size

File: src/intellwheels_desc/urdf/base.urdf.xacro (robot description, xacro)
@@ -2,12 +2,11 @@
 <robot xmlns:xacro="http://www.ros.org/wiki/xacro">
 	<xacro:macro name="base">
-		<xacro:property name="height" value="0.56"/>
-		<xacro:property name="origin">
-			<origin xyz="0 0 ${-height / 2}"/>
-		</xacro:property>
+		<xacro:property name="dimX" value="0.45"/> <!-- sem as rodas -->
+		<xacro:property name="dimY" value="1.30"/> <!-- com as rodas pequenas -->
+		<xacro:property name="dimZ" value="1.00"/> <!-- sem o apoio da cabeca -->
+		<xacro:property name="height" value="0.17"/> <!-- A origem da base.dae esta' no meio dos centros das rodas grandes-->
 		<link name="base_footprint"/>
 		<link name="base_link">
 			<inertial>
-				<xacro:insert_block name="origin"/>
 				<mass value="145"/>
 				<inertia
@@ -17,19 +16,19 @@
 			</inertial>
 			<visual>
-				<xacro:insert_block name="origin"/>
+				<origin rpy="0 0 ${-PI/2}" />
 				<geometry>
-					<mesh filename="package://intellwheels_desc/meshes/base.dae" scale="0.25952 0.24638 0.17893"/>
+					<mesh filename="package://intellwheels_desc/meshes/base.dae"/>
 				</geometry>
 			</visual>
 			<collision>
-				<origin xyz="-0.1 -0.02 0.65" rpy="0 -0.2 0"/>
+				<origin xyz="0 0 ${dimZ/1.7}" rpy="0.2 0 ${-PI/2}"/>
 				<geometry>
-					<box size="1 1.2 1.4"/>
+					<box size="${dimX} ${dimY*0.6} ${dimZ/1.3}"/>
 				</geometry>
 			</collision>
 			<collision>
-				<origin xyz="0.59 0 -0.35" rpy="0 -0.1 0"/>
+				<origin xyz="${dimX/1.2} 0 0.08" rpy="0 0 ${-PI/2}"/>
 				<geometry>
-					<box size="0.25 0.4 0.2"/>
+					<box size="0.6 0.6 0.25"/>
 				</geometry>
 			</collision>

File: src/intellwheels_desc/urdf/caster_arm.urdf.xacro (robot description, xacro)
@@ -4,22 +4,17 @@
 		<xacro:property name="left" value="${1 - right}"/>
 		<xacro:property name="front" value="${1 - back}"/>
-		<xacro:property name="origin">
-			<origin xyz="-0.035 0 -0.04"/>
-		</xacro:property>
 		<link name="${prefix}_caster_arm_link">
 			<inertial>
-				<xacro:insert_block name="origin"/>
 				<mass value="0.5"/>
 				<xacro:insert_block name="default_inertia"/>
 			</inertial>
 			<visual>
-				<xacro:insert_block name="origin"/>
 				<geometry>
-					<mesh filename="package://intellwheels_desc/meshes/caster_arm.dae" scale="0.00951 0.00951 0.1731"/>
+					<mesh filename="package://intellwheels_desc/meshes/caster_arm.dae"/>
 				</geometry>
 			</visual>
 		</link>
 		<joint name="${prefix}_caster_arm_joint" type="continuous">
-			<origin xyz="${front * 0.435 - back * 0.485} ${left * 0.3 - right * 0.32} -0.24"/>
+			<origin xyz="${front * 0.35 - back * 0.392} ${left * 0.196 - right * 0.21} 0.122" rpy="0 0 ${-PI/2}" />
 			<parent link="base_link"/>
 			<child link="${prefix}_caster_arm_link"/>

File: src/intellwheels_desc/urdf/caster_wheel.urdf.xacro (robot description, xacro)
@@ -5,5 +5,5 @@
 		<xacro:property name="front" value="${1 - back}"/>
 		<xacro:property name="origin">
-			<origin rpy="0 0 ${right * PI}"/>
+			<origin rpy="0 0 ${left * PI}"/>
 		</xacro:property>
 		<link name="${prefix}_caster_wheel_link">
@@ -16,19 +16,19 @@
 				<xacro:insert_block name="origin"/>
 				<geometry>
-					<mesh filename="package://intellwheels_desc/meshes/wheel.dae" scale="0.01306 0.01306 0.01306"/>
+					<mesh filename="package://intellwheels_desc/meshes/wheel.dae" scale="0.5 0.5 0.5"/>
 				</geometry>
 			</visual>
 			<collision>
-				<origin rpy="${PI / 2} 0 0"/>
+				<origin rpy="${PI / 2} 0 ${PI/2 - PI*right}"/>
 				<geometry>
-					<cylinder radius="0.115" length="0.1"/>
+					<cylinder radius="0.09" length="0.05"/>
 				</geometry>
 			</collision>
 		</link>
 		<joint name="${prefix}_caster_wheel_joint" type="continuous">
-			<origin xyz="-0.065 0 -0.2" rpy="0 0 ${front * PI}"/>
+			<origin xyz="0.0025 -0.044 -0.216" />
 			<parent link="${prefix}_caster_arm_link"/>
 			<child link="${prefix}_caster_wheel_link"/>
-			<axis xyz="0 1 0"/>
+			<axis xyz="1 0 0"/>
 		</joint>
 	</xacro:macro>

File: src/intellwheels_desc/urdf/diff_drive.gazebo.xacro (robot description, xacro)
@@ -1,5 +1,5 @@
 <?xml version="1.0"?>
 <robot xmlns:xacro="http://www.ros.org/wiki/xacro">
-	<xacro:macro name="diff_drive_controller">
+	<xacro:macro name="diff_drive_controller" params="pub_odom:=true">
 		<gazebo>
 			<plugin name="differential_drive_controller" filename="libgazebo_ros_diff_drive.so">
@@ -7,6 +7,6 @@
 				<leftJoint>left_drive_wheel_joint</leftJoint>
 				<rightJoint>right_drive_wheel_joint</rightJoint>
-				<wheelSeparation>0.78</wheelSeparation>
-				<wheelDiameter>0.42</wheelDiameter>
+				<wheelSeparation>0.572</wheelSeparation>
+				<wheelDiameter>0.368</wheelDiameter>
 				<wheelAcceleration>1</wheelAcceleration>
 				<wheelTorque>20</wheelTorque>
@@ -17,9 +17,9 @@
 				<odometrySource>world</odometrySource>
 				<publishWheelTF>false</publishWheelTF>
-				<publishOdomTF>true</publishOdomTF>
+				<publishOdomTF>${pub_odom}</publishOdomTF>
+				<publishTf>${pub_odom}</publishTf>
 				<publishWheelJointState>false</publishWheelJointState>
 				<legacyMode>false</legacyMode>
 				<rosDebugLevel>na</rosDebugLevel>
-				<publishTf>true</publishTf>
 			</plugin>
 		</gazebo>

File: src/intellwheels_desc/urdf/drive_wheel.urdf.xacro (robot description, xacro)
@@ -5,5 +5,5 @@
 		<xacro:property name="front" value="${1 - back}"/>
 		<xacro:property name="origin">
-			<origin rpy="0 0 ${right * PI}"/>
+			<origin xyz="0 0 -0.005" rpy="0 0 ${PI / 2 - right * PI}" />
 		</xacro:property>
 		<link name="${prefix}_drive_wheel_link">
@@ -16,5 +16,5 @@
 				<xacro:insert_block name="origin"/>
 				<geometry>
-					<mesh filename="package://intellwheels_desc/meshes/wheel.dae" scale="0.024 0.024 0.024"/>
+					<mesh filename="package://intellwheels_desc/meshes/wheel.dae"/>
 				</geometry>
 			</visual>
@@ -22,10 +22,10 @@
 				<origin rpy="${PI / 2} 0 0"/>
 				<geometry>
-					<cylinder radius="0.21" length="0.1"/>
+					<cylinder radius="0.184" length="0.07"/>
 				</geometry>
 			</collision>
 		</link>
 		<joint name="${prefix}_drive_wheel_joint" type="continuous">
-			<origin xyz="0 ${left * 0.38 - right * 0.4} -0.345"/>
+			<origin xyz="0 ${left * 0.294 - right * 0.278} 0"/>
 			<parent link="base_link"/>
 			<child link="${prefix}_drive_wheel_link"/>

File: src/intellwheels_desc/urdf/realsense.urdf.xacro (robot description, xacro)
@@ -27,5 +27,5 @@
 		</link>
 		<joint name="realsense_support_joint" type="fixed">
-			<origin xyz="-0.6 0 1.15" rpy="0 0.2 0"/>
+			<origin xyz="-0.4 0 0.9" rpy="0 0.1 0"/>
 			<parent link="base_link"/>
 			<child link="realsense_support_link"/>

File: src/intellwheels_desc/urdf/rplidar.gazebo.xacro (robot description, xacro)
@@ -1,8 +1,12 @@
 <?xml version="1.0"?>
 <robot xmlns:xacro="http://www.ros.org/wiki/xacro">
-	<xacro:macro name="rplidar_sensor" params="prefix">
+	<xacro:macro name="rplidar_sensor" params="prefix right:=0 back:=0">
+		<xacro:property name="left" value="${1 - right}"/>
+		<xacro:property name="front" value="${1 - back}"/>
+		<xacro:property name="front_angle_calib" value="${0.075*PI}"/>
+		<xacro:property name="back_angle_calib" value="0"/>
 		<gazebo reference="${prefix}_rplidar_link">
 			<sensor name="${prefix}_rplidar" type="ray">
-				<visualize>false</visualize>
+				<visualize>true</visualize>
 				<update_rate>30</update_rate>
 				<ray>
@@ -11,11 +15,11 @@
 							<samples>720</samples>
 							<resolution>1</resolution>
-							<min_angle>${-PI / 2}</min_angle>
-							<max_angle>${PI / 2}</max_angle>
+							<min_angle>${ -front * front_angle_calib -back*back_angle_calib }</min_angle>
+							<max_angle>${ 3/2*PI -front * front_angle_calib -back*back_angle_calib }</max_angle>
 						</horizontal>
 					</scan>
 					<range>
 						<min>0.20</min>
-						<max>25</max>
+						<max>15</max>
 						<resolution>0.01</resolution>
 					</range>

File: src/intellwheels_desc/urdf/rplidar.urdf.xacro (robot description, xacro)
@@ -4,15 +4,12 @@
 		<xacro:property name="left" value="${1 - right}"/>
 		<xacro:property name="front" value="${1 - back}"/>
-		<xacro:property name="origin">
-			<origin rpy="0 0 ${PI}"/>
-		</xacro:property>
+		<xacro:property name="front_angle_calib" value="${0.075*PI}"/>
+		<xacro:property name="back_angle_calib" value="0"/>
 		<link name="${prefix}_rplidar_link">
 			<inertial>
-				<xacro:insert_block name="origin"/>
 				<mass value="1"/>
 				<xacro:insert_block name="default_inertia"/>
 			</inertial>
 			<visual>
-				<xacro:insert_block name="origin"/>
 				<geometry>
 					<mesh filename="package://intellwheels_desc/meshes/rplidar.dae"/>
@@ -22,6 +19,6 @@
 		<joint name="${prefix}_rplidar_joint" type="fixed">
 			<origin
-				xyz="${front * 0.435 - back * 0.485} ${left * 0.3 - right * 0.32} -0.15"
-				rpy="0 0 ${back * PI}"/>
+				xyz="${front * 0.578 - back * 0.377} ${back * 0.245 - front * 0.235} ${back*(0.41-0.17) + front*(0.41-0.17)}"
+				rpy="0 0 ${front*(PI + front_angle_calib) + back*(0+back_angle_calib)}"/>
 			<parent link="base_link"/>
 			<child link="${prefix}_rplidar_link"/>

File: src/intellwheels_desc/urdf/wheelchair.urdf.xacro (robot description, xacro)
@@ -19,6 +19,6 @@
 	<xacro:caster prefix="left_back" back="1"/>
 	<xacro:caster prefix="right_back" right="1" back="1"/>
-	<xacro:rplidar prefix="left_front"/>
-	<xacro:rplidar prefix="right_back" right="1" back="1"/>
+	<xacro:rplidar prefix="right_front" right="1"/>
+	<xacro:rplidar prefix="left_back" back="1"/>
 	<xacro:realsense/>
 	<!-- import gazebo stuff: controllers, materials, sensors, etc... -->
@@ -28,9 +28,9 @@
 	<xacro:include filename="${urdf}/realsense.gazebo.xacro"/>
 	<!-- build gazebo stuff -->
-	<xacro:diff_drive_controller/>
+	<xacro:diff_drive_controller pub_odom="true"/>
 	<xacro:drive_wheel_mat prefix="left"/>
 	<xacro:drive_wheel_mat prefix="right"/>
-	<xacro:rplidar_sensor prefix="left_front"/>
-	<xacro:rplidar_sensor prefix="right_back"/>
+	<xacro:rplidar_sensor prefix="right_front" right="1"/>
+	<xacro:rplidar_sensor prefix="left_back" back="1"/>
 	<xacro:realsense_sensor/>
 </robot>
